Commit message: fixed the wheel display bug;add camera xacro file and add it to tank model

File: src/tank_model/urdf/tank_model.xacro (robot description, xacro)
@@ -2,4 +2,5 @@
 <robot name="tank_model" xmlns:xacro="http://www.ros.org/wiki/xacro">
     <xacro:include filename="$(find tank_model)/urdf/wheel_gazebo.xacro" />
+    <xacro:include filename="$(find tank_model)/urdf/camera_gazebo.xacro"/>
     <xacro:macro name="wheel_joint" params="prefix lr_reflect fb_reflect">
         <joint name="${prefix}_wheel_joint" type="continuous">
@@ -24,18 +25,8 @@
         <origin xyz="0.2 0 0.025" rpy="0 0 0"/>
         <parent link="base_link"/>
-        <child link="tank_camera_link"/>
+        <child link="front_camera_link"/>
         <axis xyz="0 1 0"/>
     </joint>
-    <link name="tank_camera_link">
-        <visual>
-            <origin xyz=" -0.0125 0 0.015" rpy="0 0 0" />
-            <geometry>
-                <box size="0.025 0.1 0.03" />
-            </geometry>
-            <material name="green">
-                <color rgba="0 1 0 1"/>
-            </material>
-        </visual>
-    </link>
+    <xacro:usb_camera prefix="front_camera"/>
     <joint name="tank_body_joint" type="fixed">
         <origin xyz="-0.05 0 0.025" rpy="0 0 0"/>

File: src/tank_model/urdf/wheel_gazebo.xacro (robot description, xacro)
@@ -1,5 +1,5 @@
 <?xml version="1.0"?>
 <robot xmlns:xacro="http://www.ros.org/wiki/xacro" name="wheel">
-    <xacro:property name="M_PI" value="3.1415926"/>
+    <xacro:include filename="$(find tank_model)/urdf/common_gazebo.xacro"/>
     <xacro:property name="wheel_mass" value="0.2"/>
     <xacro:property name="wheel_radius" value="0.06"/>
@@ -22,11 +22,5 @@
                 </geometry>
             </collision>
-            <!-- enable this inertial lable will not show the wheel model, the err str is 'iyy is not a valid double', why? -->
-            <!-- <inertial>
-                <mass value="${wheel_mass}"/>
-                <inertia ixx="${wheel_mass*(3*wheel_radius*wheel_radius+wheel_length*wheel_length)/12}"
-                            ixy="0" ixz="0" iyy="{wheel_mass*(3*wheel_radius*wheel_radius+wheel_length*wheel_length)/12}"
-                            iyz="0" izz="${wheel_mass*wheel_radius*wheel_radius/2}"/>
-            </inertial> -->
+            <xacro:cylinder_inertial_matrix m="${wheel_mass}" r="${wheel_radius}" h="${wheel_length}"/>
         </link>
         <gazebo reference="${prefix}_wheel_link">
