Commit message: add worlds dir and base world model;now load model to gazebo can work, and it's camera can use by rqt image display function

File: src/tank_model/urdf/camera_gazebo.xacro (robot description, xacro)
@@ -46,5 +46,5 @@
                     </noise>
                 </camera>
-                    <plugin name="gazebo_camera" filename="libgazebo_ros_camera.so">
+                <plugin name="gazebo_camera" filename="libgazebo_ros_camera.so">
 				    <ros>
 				        <!-- <namespace>stereo</namespace> -->

File: src/tank_model/urdf/tank_model.xacro (robot description, xacro)
@@ -63,4 +63,5 @@
         </visual>
     </link>
+macro
     <xacro:wheel_joint prefix="left_front" lr_reflect="1" fb_reflect="1"/>
     <xacro:wheel prefix="left_front"/>
@@ -71,3 +72,23 @@
     <xacro:wheel_joint prefix="right" lr_reflect="-1" fb_reflect="-1"/>
     <xacro:wheel prefix="right"/>
+    <gazebo>
+        <plugin name="differential_drive_controller"
+                filename="libgazebo_ros_diff_drive.so">
+                <update_rate>30</update_rate>
+                <left_joint>left_front_wheel_joint</left_joint>
+                <right_joint>right_front_wheel_joint</right_joint>
+                <wheel_separation>${wheel_joint_y*2}</wheel_separation>
+                <wheel_diameter>${2*wheel_radius}</wheel_diameter>
+                <max_wheel_torque>20</max_wheel_torque>
+                <max_wheel_acceleration>1.0</max_wheel_acceleration>
+                <command_topic>cmd_vel</command_topic>
+                <publish_odom>true</publish_odom>
+                <publish_odom_tf>true</publish_odom_tf>
+                <publish_wheel_tf>true</publish_wheel_tf>
+                <odometry_topic>odom</odometry_topic>
+                <odometry_frame>odom</odometry_frame>
+                <robot_base_frame>base_footprint</robot_base_frame>
+                <odometry_source>1</odometry_source>
+        </plugin>
+    </gazebo>
 </robot>

File: src/tank_model/urdf/wheel_gazebo.xacro (robot description, xacro)
@@ -5,4 +5,5 @@
     <xacro:property name="wheel_radius" value="0.06"/>
     <xacro:property name="wheel_length" value="0.025"/>
+    <xacro:property name="wheel_joint_y" value="0.19"/>
     <xacro:macro name="wheel" params="prefix">
         <link name="${prefix}_wheel_link">
@@ -12,5 +13,5 @@
                     <cylinder radius="${wheel_radius}" length="${wheel_length}"/>
                 </geometry>
-                <material name="white">
+                <material name="Gray">
                     <color rgba="1 1 1 0.9"/>
                 </material>
@@ -24,7 +25,7 @@
             <xacro:cylinder_inertial_matrix m="${wheel_mass}" r="${wheel_radius}" h="${wheel_length}"/>
         </link>
-        <gazebo reference="${prefix}_wheel_link">
+        <!-- <gazebo reference="${prefix}_wheel_link">
             <material>Gazebo/Gray</material>
-        </gazebo>
+        </gazebo> -->
         <transmission name="${prefix}_wheel_joint_trans">
             <type>transmission_interface/SimpleTransmission</type>
